File: hardware/stm32-peri.kicad_sch (KiCad schematic)
At the start: 64 parts, among them IC1 STM32WLE5CCU6, J1 SMA, U1 SKY13373-460LF, U2 BALFHB-WL-02D3, U3 SN74LVC1G3157DBVR, Y1 ABS07L-32.768KHZ-T, Y2 ASTX-H11

Commit message: schematic update and pcb route v1
Parts:
- removed C12: .47u, Capacitor_SMD:C_0805_2012Metric, symbol Device:C
- removed C13: 100n, Capacitor_SMD:C_0805_2012Metric, symbol Device:C
- removed C16: 100p, Capacitor_SMD:C_0402_1005Metric, symbol Device:C
- removed C17: 8p, Capacitor_SMD:C_0402_1005Metric, symbol Device:C
- removed C18: 0.7p, Capacitor_SMD:C_0402_1005Metric, symbol Device:C
- removed C19: 3p, Capacitor_SMD:C_0402_1005Metric, symbol Device:C
- removed C20, C23: 68p, Capacitor_SMD:C_0402_1005Metric, symbol Device:C
- removed C22: (no value), Capacitor_SMD:C_0402_1005Metric, symbol Device:C
- removed C44: 0.1, Capacitor_SMD:C_0805_2012Metric, symbol Device:C
- removed J1: SMA, imported-footprints:CINCH_142-0701-231, symbol imported-symbols:142-0701-231
- removed L1: L, imported-footprints:IND_BLM18KG601SN1D_MUR-M, symbol Device:L_Ferrite
- removed L2: 15u, Inductor_SMD:L_0402_1005Metric, symbol Device:L
- removed L6: 2.6n, Inductor_SMD:L_0402_1005Metric, symbol Device:L
- removed L9: L_Ferrite_Small, imported-footprints:IND_BLM18KG601SN1D_MUR-M, symbol Device:L_Ferrite_Small
- removed R4: R, Resistor_SMD:R_0805_2012Metric, symbol Device:R
- removed U2: BALFHB-WL-02D3, imported-footprints:CSPG8_STM, symbol imported-symbols:BALFHB-WL-02D3
- added BT1: Battery_Cell, Battery:BatteryHolder_Keystone_3034_1x20mm, symbol Device:Battery_Cell
- added C11: .47u, Capacitor_SMD:C_0805_2012Metric, symbol Device:C_Small
- added C27: 10p, Capacitor_SMD:C_0402_1005Metric, symbol Device:C
- added C30: 0.7p, Capacitor_SMD:C_0402_1005Metric, symbol Device:C
- added C31: 39p, Capacitor_SMD:C_0402_1005Metric, symbol Device:C
- added C32: 2p, Capacitor_SMD:C_0402_1005Metric, symbol Device:C
- added C35: 8p, Capacitor_SMD:C_0402_1005Metric, symbol Device:C
- added C37: 100p, Capacitor_SMD:C_0402_1005Metric, symbol Device:C
- added C38: 68p, Capacitor_SMD:C_0402_1005Metric, symbol Device:C
- added J5: SMA, Connector_Coaxial:SMA_Amphenol_132289_EdgeMount, symbol Connector:Conn_Coaxial
- added L1: 15u, Inductor_SMD:L_0402_1005Metric, symbol Device:L_Small
- added L2: 600R@100MHz, imported-footprints:IND_BLM18KG601SN1D_MUR-M, symbol Device:L_Ferrite
- added L3: 600R@100MHz, imported-footprints:IND_BLM18KG601SN1D_MUR-M, symbol Device:L_Ferrite_Small
- added L8: 8.7n, Inductor_SMD:L_0402_1005Metric, symbol Device:L
- added R25: R, Resistor_SMD:R_0805_2012Metric, symbol Device:R
- added U5: BALFHB-WL-05D3, imported-footprints:BGA8_BALFHB_STM, symbol imported-symbols:BALFHB-WL-05D3
- C18: renamed from C28; value 3p -> 33p
- C23: renamed from C32; footprint Capacitor_SMD:C_0805_2012Metric -> Capacitor_SMD:C_0402_1005Metric
- C24: renamed from C31; footprint Capacitor_SMD:C_0805_2012Metric -> Capacitor_SMD:C_0402_1005Metric
- C26: renamed from C33; footprint Capacitor_SMD:C_0805_2012Metric -> Capacitor_SMD:C_0402_1005Metric
- C28: renamed from C14; footprint Capacitor_SMD:C_0402_1005Metric -> Capacitor_SMD:C_0805_2012Metric
- C29: renamed from C15; footprint Capacitor_SMD:C_0402_1005Metric -> Capacitor_SMD:C_0805_2012Metric
- C33: renamed from C41; footprint Capacitor_SMD:C_0805_2012Metric -> Capacitor_SMD:C_0402_1005Metric
- C34: value 10p -> 100p; footprint Capacitor_SMD:C_0805_2012Metric -> Capacitor_SMD:C_0402_1005Metric
- C39: renamed from C40; footprint Capacitor_SMD:C_0805_2012Metric -> Capacitor_SMD:C_0402_1005Metric
- C40: renamed from C39; footprint Capacitor_SMD:C_0805_2012Metric -> Capacitor_SMD:C_0402_1005Metric
- C41: renamed from C42; footprint Capacitor_SMD:C_0805_2012Metric -> Capacitor_SMD:C_0402_1005Metric
- C42: renamed from C43; footprint Capacitor_SMD:C_0805_2012Metric -> Capacitor_SMD:C_0402_1005Metric
- C46: renamed from C21; footprint Capacitor_SMD:C_0402_1005Metric -> Capacitor_SMD:C_0805_2012Metric; now not fitted
- L7: value 10n -> 3.6n
- Y1: symbol imported-symbols:ABS07L-32.768KHZ-T -> Device:Crystal_Small
- renumbered C7 to C10, C49 to C12, C10 to C13, C11 to C14, C48 to C15, C5 to C17, C36 to C19, C35 to C20, C37 to C21, C29 to C22, C30 to C25, C24 to C36, C25 to C43, C26 to C44, C27 to C45, C1 to C5, C2 to C6, C3 to C7, C4 to C8, C6 to C9, D2 to D7, D3 to D8, L3 to L6, L8 to L9, R2 to R26, R1 to R27, U1 to U3, U3 to U4
Connections:
- net +3.3V: now also D7.2 (A), L2.1
- net GND: now also C28.1, C29.1, BT1.2 (-), C11.1, C27.2, C30.2, C35.2, C37.1, J5.2 (Ext), U5.B1 (GND2), U5.B2 (GND3), U5.C2 (GND1); no longer C28.2, C29.2, C34.2
- net VBAT: now also BT1.1 (+), R25.2; no longer D7.1 (K)
- net VDDA: now also L2.2
- net VDDRF1V55: now also C11.2, L1.2
- net VLXSMPS: now also L1.1
- net at L6.1: now also C28.2, C29.2, IC1.24 (VR_PA), L4.1; no longer IC1.23 (RFO_HP)
- net at U3.1 (J1): now also C46.1, L8.1
- net at L5.1: now also IC1.23 (RFO_HP); no longer L4.1
- net at C26.1, IC1.15 (PA7), U3.5 (V2): now also C27.1; no longer C34.1
- net at U3.3 (J3): now also C31.2
- net at C44.1, D8.2 (A2), L9.1: now also J5.1 (In)
- net at IC1.30 (PB0-VDD_TCXO): now also L3.1
- net at Y2.4 (VDD): now also L3.2
- net RFI_N: now reaches IC1.21 (RFI_N)
- net RFI_N: now also U5.A2 (RFI_N_OUT)
- net RFI_P: now reaches IC1.20 (RFI_P)
- net RFI_P: now also U5.A3 (RFI_P_OUT)
- net at L7.2: now also L5.2, L6.2, C30.1, C32.2
- net RFO_LP: no longer names the net of IC1.22 (RFO_LP)
- net RFO_LP: now also C34.2, L4.2; no longer L5.2
- removed net VR_PA: C28.1, C29.1, IC1.24 (VR_PA), L4.2, L6.2
- new net: C38.1, L8.2
- new net: C32.1, C35.1, C38.2, L7.1
- new net: C31.1, U5.C1 (RFO_OUT)
- new net: C37.2, U3.9 (J2), U5.C3 (RFI_IN)
- new net: C34.1, U5.A1 (RFO_IN)
- new net: D7.1 (K), R25.1
Other:
- note added: "RF Power Supply: Caps close to MCU"
- note removed: "RF Power Supply"
- moved on the sheet: C10, C12, C13, C14, C15, C17, C18, C28, C29, C44, C45, C5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

Commit message: better pcb route (no test pads)
Parts:
- removed C23, C26: 1n, Capacitor_SMD:C_0402_1005Metric, symbol Device:C
- removed C8: 100n, Capacitor_SMD:C_0805_2012Metric, symbol Device:C
- C10: renamed from C43; KiLib_Generator (none) -> SMD_2terminal_chip_molded
- C11: renamed from C24; value 10p -> 100p; KiLib_Generator (none) -> SMD_2terminal_chip_molded
- C12: renamed from C31; KiLib_Generator (none) -> SMD_2terminal_chip_molded
- C13: renamed from C44; KiLib_Generator (none) -> SMD_2terminal_chip_molded
- C14: renamed from C15; KiLib_Generator (none) -> SMD_2terminal_chip_molded
- C15: renamed from C27; value 10p -> 100p; KiLib_Generator (none) -> SMD_2terminal_chip_molded
- C16: renamed from C32; KiLib_Generator (none) -> SMD_2terminal_chip_molded
- C17: renamed from C38; KiLib_Generator (none) -> SMD_2terminal_chip_molded
- C18: renamed from C46; KiLib_Generator (none) -> SMD_2terminal_chip_molded
- C19: renamed from C30; KiLib_Generator (none) -> SMD_2terminal_chip_molded
- C20: renamed from C35; KiLib_Generator (none) -> SMD_2terminal_chip_molded
- C21, L1, L5, R25: KiLib_Generator (none) -> SMD_2terminal_chip_molded
- C22: renamed from C19; KiLib_Generator (none) -> SMD_2terminal_chip_molded
- C24: renamed from C20; KiLib_Generator (none) -> SMD_2terminal_chip_molded
- C25: renamed from C28; KiLib_Generator (none) -> SMD_2terminal_chip_molded
- C26: renamed from C33; KiLib_Generator (none) -> SMD_2terminal_chip_molded
- C27: renamed from C39; KiLib_Generator (none) -> SMD_2terminal_chip_molded
- C28: renamed from C17; KiLib_Generator (none) -> SMD_2terminal_chip_molded
- C29: renamed from C40; KiLib_Generator (none) -> SMD_2terminal_chip_molded
- C30: renamed from C29; KiLib_Generator (none) -> SMD_2terminal_chip_molded
- C31: renamed from C22; KiLib_Generator (none) -> SMD_2terminal_chip_molded
- C32: renamed from C42; KiLib_Generator (none) -> SMD_2terminal_chip_molded
- C33: renamed from C10; KiLib_Generator (none) -> SMD_2terminal_chip_molded
- C34: renamed from C9; KiLib_Generator (none) -> SMD_2terminal_chip_molded
- C35: renamed from C41; KiLib_Generator (none) -> SMD_2terminal_chip_molded
- C36: renamed from C25; KiLib_Generator (none) -> SMD_2terminal_chip_molded
- C37: renamed from C7; KiLib_Generator (none) -> SMD_2terminal_chip_molded
- C38: renamed from C18; KiLib_Generator (none) -> SMD_2terminal_chip_molded
- C39: renamed from C13; KiLib_Generator (none) -> SMD_2terminal_chip_molded
- C4: renamed from C11; KiLib_Generator (none) -> SMD_2terminal_chip_molded
- C40: renamed from C14; KiLib_Generator (none) -> SMD_2terminal_chip_molded
- C41: renamed from C6; KiLib_Generator (none) -> SMD_2terminal_chip_molded
- C42: renamed from C5; KiLib_Generator (none) -> SMD_2terminal_chip_molded
- C5: renamed from C37; KiLib_Generator (none) -> SMD_2terminal_chip_molded
- C6: renamed from C12; KiLib_Generator (none) -> SMD_2terminal_chip_molded
- C7: renamed from C34; KiLib_Generator (none) -> SMD_2terminal_chip_molded
- C8: renamed from C45; KiLib_Generator (none) -> SMD_2terminal_chip_molded
- C9: renamed from C36; KiLib_Generator (none) -> SMD_2terminal_chip_molded
- L2: renamed from L4; KiLib_Generator (none) -> SMD_2terminal_chip_molded
- L3: renamed from L9; KiLib_Generator (none) -> SMD_2terminal_chip_molded
- L4: renamed from L6; KiLib_Generator (none) -> SMD_2terminal_chip_molded
- L6: renamed from L7; KiLib_Generator (none) -> SMD_2terminal_chip_molded
- L7: renamed from L8; KiLib_Generator (none) -> SMD_2terminal_chip_molded
- R20: renamed from R26; KiLib_Generator (none) -> SMD_2terminal_chip_molded
- R24: renamed from R27; KiLib_Generator (none) -> SMD_2terminal_chip_molded
- renumbered D8 to D5, D7 to D8, J5 to J4, L3 to L8, L2 to L9, IC1 to MCU1, U5 to U3, U3 to U4, U4 to U5
Connections:
- net GND: no longer C14.2, C21.2, C24.2, C6.2, Y2.2 (GND)
- net OSC_K-: now reaches C14.1, MCU1.39 (PC14-OSC32_IN), Y1.1
- net OSC_K+: now reaches C6.1, MCU1.40 (PC15-OSC32_OUT), Y1.2
- net at C15.1, MCU1.15 (PA7): now also U4.4 (V1); no longer U4.5 (V2)
- net at C11.1, MCU1.14 (PA6): now also U4.5 (V2); no longer U4.4 (V1)
- new net GND1: C14.2, C21.2, C24.2, C6.2, Y2.2 (GND)

Commit message: pcb v2 update: test points, stickers, labeling
Parts:
- added C43: 8p, Capacitor_SMD:C_0402_1005Metric, symbol Device:C
- added L10: 3.6n, Inductor_SMD:L_0402_1005Metric, symbol Device:L
- added R28, R29: R_Small_US, Resistor_SMD:R_0201_0603Metric_Pad0.64x0.40mm_HandSolder, symbol Device:R_Small_US
- C18: footprint Capacitor_SMD:C_0805_2012Metric -> Capacitor_SMD:C_0402_1005Metric
- C5: now not fitted
Connections:
- net GND: now also C43.2
- net RFI_N: now also R29.2; no longer MCU1.21 (RFI_N)
- net RFI_P: now also R28.2; no longer MCU1.20 (RFI_P)
- net at C5.2, U3.C3 (RFI_IN): now also L10.2; no longer U4.9 (J2)
- new net: C43.1, L10.1, U4.9 (J2)
- new net mcuRFI_N: MCU1.21 (RFI_N), R29.1
- new net mcuRFI_P: MCU1.20 (RFI_P), R28.1
Other:
- moved on the sheet: C9
